File: Pyxel-Paradise.sch (KiCad schematic (older format))
At the start: 33 parts, among them J1 Joystick-North, J10 Action-Up, J11 Action-Right, J12 Action-Down, J13 Action-Left, J14 Meta-Button-1, J15 Meta-Button-2, J16 Meta-Button-3, J17 Meta-Button-4, J2 Joystick-NorthEast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

Commit message: V1 of a working PCB is complete
Parts:
- removed J1: Joystick-North, Connector_JST:JST_XH_B02B-XH-A_1x02_P2.50mm_Vertical, symbol Connector_Generic:Conn_01x02
- removed J2: Joystick-NorthEast, Connector_JST:JST_XH_B02B-XH-A_1x02_P2.50mm_Vertical, symbol Connector_Generic:Conn_01x02
- removed J3: Joystick-East, Connector_JST:JST_XH_B02B-XH-A_1x02_P2.50mm_Vertical, symbol Connector_Generic:Conn_01x02
- removed J4: Joystick-SouthEast, Connector_JST:JST_XH_B02B-XH-A_1x02_P2.50mm_Vertical, symbol Connector_Generic:Conn_01x02
- removed J5: Joystick-South, Connector_JST:JST_XH_B02B-XH-A_1x02_P2.50mm_Vertical, symbol Connector_Generic:Conn_01x02
- removed J6: Joystick-SouthWest, Connector_JST:JST_XH_B02B-XH-A_1x02_P2.50mm_Vertical, symbol Connector_Generic:Conn_01x02
- removed J7: Joystick-West, Connector_JST:JST_XH_B02B-XH-A_1x02_P2.50mm_Vertical, symbol Connector_Generic:Conn_01x02
- removed J8: Joystick-NorthWest, Connector_JST:JST_XH_B02B-XH-A_1x02_P2.50mm_Vertical, symbol Connector_Generic:Conn_01x02
- removed J9: Raspberry_Pi_2_3, Connector_PinHeader_2.54mm:PinHeader_2x20_P2.54mm_Vertical, symbol Connector:Raspberry_Pi_2_3
- removed R13, R14, R15, R16: 10k, Resistor_THT:R_Axial_DIN0207_L6.3mm_D2.5mm_P2.54mm_Vertical, symbol Device:R
- added J1: Conn_01x05, Connector_JST:JST_XH_B05B-XH-A_1x05_P2.50mm_Vertical, symbol Connector_Generic:Conn_01x05
- added U1: Arduino_ProMicro_Socket, Arduino:Aruduino_ProMicro_Socket, symbol arduino:Arduino_ProMicro_Socket
Connections:
- net labels added: JOYSTICK_EAST, JOYSTICK_NORTH, JOYSTICK_SOUTH, JOYSTICK_WEST, VCC
- net labels removed: +3.3V, East, North, NorthEast, NorthWest, South, SouthEast, SouthWest, West
- wire segments 98 -> 66
Other:
- moved on the sheet: J10, J11, J12, J13, J14, J15, J16, J17, R1, R2, R3, R4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
